Commit message: Add simple model

File: workspace/src/my_package/description/sliding_robot_arm_with_cam.urdf.xacro (robot description, xacro)
@@ -125,5 +125,5 @@
         </collision>
         <xacro:inertial_box mass="0.1" x="0.12" y="0.15" z="0.15">
-            <oeigin xyz="0 0 0" rpy="0 0 0" />
+            <origin xyz="0 0 0" rpy="0 0 0" />
         </xacro:inertial_box>
     </link>
